Commit message: added easynav

File: robot_description/urdf/robot_gazebo_control.xacro (robot description, xacro)
@@ -1,5 +1,5 @@
 <?xml version="1.0"?>
 <robot xmlns:xacro="http://ros.org/wiki/xacro">
-  <gazebo reference="chassis">
+  <gazebo reference="base_link">
     <visual>
       <xacro:gz_material_orange/>
@@ -51,5 +51,5 @@
       <odom_topic>odom</odom_topic>
       <odom_frame>odom</odom_frame>
-      <robot_base_frame>base_link</robot_base_frame>
+      <robot_base_frame>base_footprint</robot_base_frame>
       <publish_tf>true</publish_tf>
       <tf_topic>tf</tf_topic>

File: robot_description/urdf/robot_urdf.xacro (robot description, xacro)
@@ -65,12 +65,12 @@
     <xacro:include filename="$(find robot_description)/urdf/robot_gazebo_properties.xacro" />
     <xacro:include filename="$(find robot_description)/urdf/robot_gazebo_control.xacro" />
-    <link name="base_link">
+    <link name="base_footprint">
     </link>
     <joint name="chassis_joint" type="fixed">
-        <parent link="base_link"/>
-        <child link="chassis"/>
+        <parent link="base_footprint"/>
+        <child link="base_link"/>
         <origin xyz="0 0 ${wheel_radius+wheel_height_offset}"/>
     </joint>
-    <link name="chassis">
+    <link name="base_link">
         <xacro:insert_box_with_fillet x="-0.040" y="0" z="0"
             size_x="${chassis_length}" size_y="${chassis_width}" size_z="${slab_height}"
@@ -120,5 +120,5 @@
         base_name="left_wheel"
         parent_name="base_link"
-        x="0" y="${wheel_seperation/2}" z="${wheel_radius}"
+        x="0" y="${wheel_seperation/2}" z="${-wheel_height_offset}"
         mass="${wheel_mass}"
         radius="${wheel_radius}"
@@ -133,5 +133,5 @@
         base_name="right_wheel"
         parent_name="base_link"
-        x="0" y="${-wheel_seperation/2}" z="${wheel_radius}"
+        x="0" y="${-wheel_seperation/2}" z="${-wheel_height_offset}"
         mass="${wheel_mass}"
         radius="${wheel_radius}"
@@ -146,5 +146,5 @@
         <parent link="base_link"/>
         <child link="castor_wheel"/>
-        <origin xyz="-0.10 0 ${castor_wheel_diameter/2}"/>
+        <origin xyz="-0.10 0 ${-castor_wheel_diameter/2}"/>
     </joint>
     <link name="castor_wheel">
@@ -171,9 +171,9 @@
     <xacro:insert_lidar
         base_name="lidar"
-        parent_name="chassis"
+        parent_name="base_link"
         x="-0.0115" y="0" z="${chassis_height+lidar_z_offset}"
         mass="0.1"/>
     <joint name="imu_joint" type="fixed">
-        <parent link="chassis"/>
+        <parent link="base_link"/>
         <child link="imu"/>
         <origin xyz="0.03 0 ${chassis_height}"/>
